Commit message: fix: fixed realsense urdf

File: src/orion_vi_description/urdf/bootlegsense.urdf.xacro (robot description, xacro)
@@ -2,45 +2,28 @@
 <robot xmlns:xacro="http://www.ros.org/wiki/xacro" >
 <xacro:macro name="add_realsense_link" params="suffix">
-    <link name="realsense_${suffix}_link">
-      <inertial>
-        <mass>0.0615752</mass>
-        <inertia>
-          <ixx>9.108e-05</ixx>
-          <ixy>0</ixy>
-          <ixz>0</ixz>
-          <iyy>2.51e-06</iyy>
-          <iyz>0</iyz>
-          <izz>8.931e-05</izz>
-        </inertia>
-        <pose frame=''>0 0 0 0 -0 0</pose>
-      </inertial>
-      <collision name="collision">
-        <geometry>
-          <mesh filename="meshes/realsense.dae"/>
-        </geometry>
-      </collision>
-      <visual name= "visual">
-        <geometry>
-          <mesh filename="meshes/realsense.dae">
-          <submesh>
-              <name>RealSense</name>
-              <center>false</center>
-          </submesh>
-          </mesh>
-        </geometry>
-        <material>
-          <diffuse>1.0 1.0 1.0</diffuse>
-          <specular>1.0 1.0 1.0</specular>
-          <pbr>
-            <metal>
-              <albedo_map>sensors/RealSense_D435/materials/textures/RealSense_Albedo.png</albedo_map>
-              <normal_map>sensors/RealSense_D435/materials/textures/RealSense_Normal.png</normal_map>
-              <metalness_map>sensors/RealSense_D435/materials/textures/RealSense_Metalness.png</metalness_map>
-              <roughness_map>sensors/RealSense_D435/materials/textures/RealSense_Roughness.png</roughness_map>
-            </metal>
-          </pbr>
-        </material>
-      </visual>
-    </link>
+  <xacro:property name="realsense_size" value="0.025 0.09 0.025"/>
+  <xacro:property name="realsense_origin" value="${chassis_x/2} 0 ${chassis_z*2}"/>
+  <material name="realsense_mat">
+      <color rgba="0.1490196 0.1490196 0.1490196 1.0"/>
+  </material>
+  <link name="realsense_${suffix}_link">
+    <inertial>
+      <mass value="0.0615752"/>
+      <inertia ixx="9.108e-05" ixy="0" ixz="0" iyy="2.51e-06" iyz="0" izz="8.931e-05"/>
+    </inertial>
+    <collision name="realsense_collision">
+      <origin xyz="${realsense_origin}"/>
+      <geometry>
+        <box size="${realsense_size}"/>
+      </geometry>
+    </collision>
+    <visual name= "realsense_visual">
+      <material name="realsense_mat"/>
+      <origin xyz="${realsense_origin}"/>
+      <geometry>
+        <box size="${realsense_size}"/>
+      </geometry>
+    </visual>
+  </link>
 </xacro:macro>
 </robot>
