Commit message: feat: added a Realsense camera therover model

File: src/orion_vi_description/urdf/orionVI.gazebo.xacro (robot description, xacro)
@@ -12,6 +12,8 @@
     </gazebo>
     <xacro:include filename="$(find orion_vi_description)/urdf/sensors/imu.xacro" />
-    <xacro:add_imu link="camera" name="camera_imu"/>
+    <xacro:add_imu link="realsense_front_link" name="realsense_front_imu"/>
     <xacro:add_imu link="left_subchassis" name="left_imu"/>
     <xacro:add_imu link="right_subchassis" name="right_imu"/>
+    <xacro:include filename="$(find orion_vi_description)/urdf/sensors/bootlegsense.xacro" />
+    <xacro:add_realsense suffix="front"/>
 </robot>

File: src/orion_vi_description/urdf/orionVI_description.urdf.xacro (robot description, xacro)
@@ -1,5 +1,5 @@
 <?xml version="1.0"?>
 <robot name="orionVI" xmlns:xacro="http://ros.org/wiki/xacro" author="Aleksandra Grzybek">
-  <!-- Converted from rover_model.sdf -->
+  <xacro:include filename="$(find orion_vi_description)/urdf/bootlegsense.urdf.xacro" />
   <!-- Properties -->
   <xacro:property name="wheel_radius" value="0.21"/>
@@ -62,15 +62,6 @@
     <color rgba="0.6431373 0.6431373 0.6431373 1.0"/>
   </material>
-  <!--CAMERA-->
-  <link name="camera">
-    <origin xyz="${chassis_x/2} 0 ${(chassis_z+chassis_origin_z)/2}" rpy="0 0 0"/>
-    <visual name="camera_visual">
-      <material name="chassis_mat"/>
-      <origin xyz="${chassis_x/2} 0 ${(chassis_z+chassis_origin_z)/2}" rpy="0 0 0"/>
-      <geometry>
-        <box size="0.1 0.2 0.1"/>
-      </geometry>
-    </visual>
-  </link>
+  <!--REALSENSE-->
+  <xacro:add_realsense_link suffix ="front"/>
   <!-- CHASSIS -->
   <link name="chassis">
@@ -270,6 +261,6 @@
 </link>
 <!-- JOINTS -->
-<joint name="camera_joint" type="fixed">
-  <parent link="camera"/>
+<joint name="realsense_front_joint" type="fixed">
+  <parent link="realsense_front_link"/>
   <child link="chassis"/>
   <axis xyz="1 0 0"/>

File: src/orion_vi_description/urdf/sensors/imu.xacro (robot description, xacro)
@@ -4,4 +4,5 @@
     <gazebo reference="${link}">
     <sensor name="${name}" type="imu">
+        <topic>${name}</topic>
         <always_on>true</always_on>
         <update_rate>100</update_rate>
@@ -48,11 +49,4 @@
           </linear_acceleration>
         </imu>
-        <plugin name="bytes_imu" filename="libgazebo_ros_imu_sensor.so">
-            <ros>
-                <namespace>imu</namespace>
-                <remapping>~/out:=data</remapping>
-            </ros>
-            <initial_orientation_as_reference>false</initial_orientation_as_reference>
-        </plugin>
     </sensor>
     </gazebo>

Commit message: feat: addded a new fancy Gazebo rover model

File: src/orion_vi_description/urdf/orionVI.gazebo.xacro (robot description, xacro)
@@ -12,8 +12,8 @@
     </gazebo>
     <xacro:include filename="$(find orion_vi_description)/urdf/sensors/imu.xacro" />
-    <xacro:add_imu link="realsense_front_link" name="realsense_front_imu"/>
-    <xacro:add_imu link="left_subchassis" name="left_imu"/>
-    <xacro:add_imu link="right_subchassis" name="right_imu"/>
+    <xacro:add_imu link="realsense" name="realsense_front_imu"/>
+    <xacro:add_imu link="rocker_L" name="left_imu"/>
+    <xacro:add_imu link="rocker_R" name="right_imu"/>
     <xacro:include filename="$(find orion_vi_description)/urdf/sensors/bootlegsense.xacro" />
-    <xacro:add_realsense suffix="front"/>
+    <xacro:add_realsense />
 </robot>

File: src/orion_vi_description/urdf/orionVI.ros2_control.xacro (robot description, xacro)
@@ -14,6 +14,6 @@
         </xacro:unless>
       </hardware>
-      <xacro:macro name="turntable" params="prefix topic_state topic_com">
-        <joint name="${prefix}_turntable_joint">
+      <xacro:macro name="turntable" params="suffix topic_state topic_com">
+        <joint name="turntable_${suffix}_joint">
           <command_interface name="position">
             <param name="topic">${topic_com}</param>
@@ -24,6 +24,6 @@
         </joint>
       </xacro:macro>
-      <xacro:macro name="wheel" params="prefix topic_state topic_com">
-        <joint name="${prefix}_wheel_joint">
+      <xacro:macro name="wheel" params="suffix topic_state topic_com">
+        <joint name="wheel_${suffix}_joint">
           <command_interface name="velocity">
             <param name="topic">${topic_com}</param>
@@ -34,12 +34,12 @@
         </joint>
       </xacro:macro>
-      <xacro:wheel prefix="left_front" topic_state="/left_front_wheel/state" topic_com="/left_front_wheel/com"/>
-      <xacro:wheel prefix="left_rear" topic_state="/left_rear_wheel/state" topic_com="/left_rear_wheel/com"/>
-      <xacro:wheel prefix="right_front" topic_state="/right_front_wheel/state" topic_com="/right_front_wheel/com"/>
-      <xacro:wheel prefix="right_rear" topic_state="/right_rear_wheel/state" topic_com="/right_rear_wheel/com"/>
-      <xacro:turntable prefix="left_front" topic_state="/left_front_turntable/state" topic_com="/left_front_turntable/com"/>
-      <xacro:turntable prefix="left_rear" topic_state="/left_rear_turntable/state" topic_com="/left_rear_turntable/com"/>
-      <xacro:turntable prefix="right_front" topic_state="/right_front_turntable/state" topic_com="/right_front_turntable/com"/>
-      <xacro:turntable prefix="right_rear" topic_state="/right_rear_turntable/state" topic_com="/right_rear_turntable/com"/>
+      <xacro:wheel suffix="F_L" topic_state="/left_front_wheel/state" topic_com="/left_front_wheel/com"/>
+      <xacro:wheel suffix="R_L" topic_state="/left_rear_wheel/state" topic_com="/left_rear_wheel/com"/>
+      <xacro:wheel suffix="F_R" topic_state="/right_front_wheel/state" topic_com="/right_front_wheel/com"/>
+      <xacro:wheel suffix="R_R" topic_state="/right_rear_wheel/state" topic_com="/right_rear_wheel/com"/>
+      <xacro:turntable suffix="F_L" topic_state="/left_front_turntable/state" topic_com="/left_front_turntable/com"/>
+      <xacro:turntable suffix="R_L" topic_state="/left_rear_turntable/state" topic_com="/left_rear_turntable/com"/>
+      <xacro:turntable suffix="F_R" topic_state="/right_front_turntable/state" topic_com="/right_front_turntable/com"/>
+      <xacro:turntable suffix="R_R" topic_state="/right_rear_turntable/state" topic_com="/right_rear_turntable/com"/>
     </ros2_control>
   </xacro:macro>

File: src/orion_vi_description/urdf/orionVI.urdf.xacro (robot description, xacro)
@@ -9,6 +9,4 @@
   <!-- Import RRBot macro -->
   <xacro:include filename="orionVI_description.urdf.xacro" />
-  <!-- Import Rviz colors -->
-  <xacro:include filename="orionVI.materials.xacro" />
   <!-- Import RRBot ros2_control description -->
   <xacro:include filename="$(find orion_vi_description)/urdf/orionVI.ros2_control.xacro" />

File: src/orion_vi_description/urdf/orionVI_description.urdf.xacro (robot description, xacro)
@@ -1,331 +1,343 @@
 <?xml version="1.0"?>
-<robot name="orionVI" xmlns:xacro="http://ros.org/wiki/xacro" author="Aleksandra Grzybek">
-  <xacro:include filename="$(find orion_vi_description)/urdf/bootlegsense.urdf.xacro" />
-  <!-- Properties -->
-  <xacro:property name="wheel_radius" value="0.21"/>
-  <xacro:property name="wheel_length" value="0.198"/>
-  <!-- Mass and geometry parameters -->
-  <xacro:property name="chassis_mass" value="20.0"/>
-  <xacro:property name="subchassis_mass" value="6.0"/>
-  <xacro:property name="wheel_mass" value="7.0"/>
-  <xacro:property name="suspension_diff_mass" value="0.001"/>
-  <xacro:property name="wheel_center_z" value="0.213"/>
-  <!-- Dimensions split into components for inertia calculation -->
-  <xacro:property name="chassis_x" value="1.055"/>
-  <xacro:property name="chassis_y" value="0.65"/>
-  <xacro:property name="chassis_z" value="0.24"/>
-  <xacro:property name="subchassis_x" value="1.0"/>
-  <xacro:property name="subchassis_y" value="0.162"/>
-  <xacro:property name="subchassis_z" value="0.06"/>
-  <!-- Inertia parameters (defaults from original SDF) -->
-  <!-- Automatic inertia calculations -->
-  <!-- temporarily use numeric literals for chassis inertia to avoid xacro eval issue -->
-  <xacro:property name="chassis_ixx" value="0.41791666666666677"/>
-  <xacro:property name="chassis_iyy" value="1.6560416666666666"/>
-  <xacro:property name="chassis_izz" value="1.4670833333333334"/>
-  <xacro:property name="subchassis_ixx" value="0.0036"/>
-  <xacro:property name="subchassis_iyy" value="0.3546"/>
-  <xacro:property name="subchassis_izz" value="0.3546"/>
-  <!-- Wheel: cylinder with axis along Y -> iyy = 1/2 m r^2; ixx=izz = 1/12 m (3 r^2 + h^2) -->
-  <xacro:property name="wheel_iyy" value="0.0929915"/>
-  <xacro:property name="wheel_ixx" value="0.0619943333333"/>
-  <xacro:property name="wheel_izz" value="${wheel_ixx}"/>
-  <!-- Suspension diff: approximate as small cube of size eps -->
-  <xacro:property name="suspdiff_dim" value="0.01"/>
-  <xacro:property name="suspdiff_ixx" value="8.33333333333e-07"/>
-  <xacro:property name="suspdiff_iyy" value="${suspdiff_ixx}"/>
-  <xacro:property name="suspdiff_izz" value="${suspdiff_ixx}"/>
-  <!-- Frame/subchassis/wheel spacing properties -->
-  <xacro:property name="chassis_size" value="${chassis_x} ${chassis_y} ${chassis_z}"/>
-  <xacro:property name="subchassis_size" value="${subchassis_x} ${subchassis_y} ${subchassis_z}"/>
-  <xacro:property name="wheel_spacing_x" value="0.9"/>
-  <xacro:property name="wheel_spacing_y" value="0.86"/>
-  <xacro:property name="wheel_subchassis_gap" value="0.02"/>
-  <!-- chassis origin height: set 0.197 m above wheel center -->
-  <xacro:property name="chassis_origin_z" value="$(eval ${wheel_center_z} + 0.197)"/>
-  <!-- subchassis origins: align tops with chassis top (subchassis top tangent to chassis top) -->
-  <xacro:property name="subchassis_origin_z" value="$(eval ${wheel_center_z} + 0.197 + ${chassis_z}/2 - ${subchassis_z}/2)"/>
-  <xacro:property name="left_subchassis_y" value="$(eval ${chassis_y}/2 + 0.01 + ${subchassis_y}/2)"/>
-  <xacro:property name="right_subchassis_y" value="$(eval -${chassis_y}/2 - 0.01 - ${subchassis_y}/2)"/>
-  <!-- turntable properties -->
-  <xacro:property name="turntable_height" value="0.10"/>
-  <xacro:property name="turntable_radius" value="$(eval ${subchassis_y}/2)"/>
-  <xacro:property name="turntable_mass" value="1.0"/>
-  <!-- Materials -->
-  <material name="wheel_mat">
-    <color rgba="0.1490196 0.1490196 0.1490196 1.0"/>
-  </material>
-  <material name="subchassis_mat">
-    <color rgba="0.3176471 0.3176471 0.3176471 1.0"/>
-  </material>
-  <material name="chassis_mat">
-    <color rgba="0.6431373 0.6431373 0.6431373 1.0"/>
-  </material>
-  <!--REALSENSE-->
-  <xacro:add_realsense_link suffix ="front"/>
-  <!-- CHASSIS -->
-  <link name="chassis">
-    <inertial>
-      <origin xyz="0 0 ${chassis_origin_z}" rpy="0 0 0"/>
-      <mass value="${chassis_mass}"/>
-      <inertia ixx="${chassis_ixx}" ixy="0" ixz="0" iyy="${chassis_iyy}" iyz="0" izz="${chassis_izz}"/>
-    </inertial>
-    <visual name="body_visual">
-      <material name="chassis_mat"/>
-      <origin xyz="0 0 ${chassis_origin_z}" rpy="0 0 0"/>
-      <geometry>
-        <box size="${chassis_x} ${chassis_y} ${chassis_z}"/>
-      </geometry>
-    </visual>
-    <collision name="body_collision">
-      <origin xyz="0 0 ${chassis_origin_z}" rpy="0 0 0"/>
-      <geometry>
-        <box size="${chassis_x} ${chassis_y} ${chassis_z}"/>
-      </geometry>
-    </collision>
-  </link>
-  <!-- LEFT SUBCHASSIS -->
-  <link name="left_subchassis">
-    <inertial>
-      <origin xyz="0 ${left_subchassis_y} ${subchassis_origin_z}" rpy="0 0 0"/>
-      <mass value="${subchassis_mass}"/>
-      <inertia ixx="${subchassis_ixx}" ixy="0" ixz="0" iyy="${subchassis_iyy}" iyz="0" izz="${subchassis_izz}"/>
-    </inertial>
-    <visual name="left_rail_visual">
-      <material name="subchassis_mat"/>
-      <origin xyz="0 ${left_subchassis_y} ${subchassis_origin_z}" rpy="0 0 0"/>
-      <geometry>
-        <box size="${subchassis_size}"/>
-      </geometry>
-    </visual>
-    <collision name="left_rail_collision">
-      <origin xyz="0 ${left_subchassis_y} ${subchassis_origin_z}" rpy="0 0 0"/>
-      <geometry>
-        <box size="${subchassis_size}"/>
-      </geometry>
-    </collision>
-  </link>
-  <!-- RIGHT SUBCHASSIS -->
-  <link name="right_subchassis">
-    <inertial>
-      <origin xyz="0 ${right_subchassis_y} ${subchassis_origin_z}" rpy="0 0 0"/>
-      <mass value="${subchassis_mass}"/>
-      <inertia ixx="${subchassis_ixx}" ixy="0" ixz="0" iyy="${subchassis_iyy}" iyz="0" izz="${subchassis_izz}"/>
-    </inertial>
-    <visual name="right_rail_visual">
-      <material name="subchassis_mat"/>
-      <origin xyz="0 ${right_subchassis_y} ${subchassis_origin_z}" rpy="0 0 0"/>
-      <geometry>
-        <box size="${subchassis_size}"/>
-      </geometry>
-    </visual>
-    <collision name="right_rail_collision">
-      <origin xyz="0 ${right_subchassis_y} ${subchassis_origin_z}" rpy="0 0 0"/>
-      <geometry>
-        <box size="${subchassis_size}"/>
-      </geometry>
-    </collision>
-  </link>
-  <!-- VIRTUAL SUSPENSION DIFF -->
-  <link name="suspension_diff">
-    <inertial>
-      <mass value="${suspension_diff_mass}"/>
-      <inertia ixx="${suspdiff_ixx}" ixy="0" ixz="0" iyy="${suspdiff_iyy}" iyz="0" izz="${suspdiff_izz}"/>
-    </inertial>
-  </link>
-  <!-- WHEELS -->
-  <link name="left_front_wheel">
-    <inertial>
-      <mass value="${wheel_mass}"/>
-      <inertia ixx="0.062" ixy="0" ixz="0" iyy="0.093" iyz="0" izz="0.062"/>
-    </inertial>
-    <visual>
-      <material name="wheel_mat"/>
-      <origin xyz="0 0 0" rpy="1.5708 0 0"/>
-      <geometry>
-        <cylinder radius="${wheel_radius}" length="${wheel_length}"/>
-      </geometry>
-    </visual>
-    <collision>
-      <origin xyz="0 0 0" rpy="1.5708 0 0"/>
-      <geometry>
-        <cylinder radius="${wheel_radius}" length="${wheel_length}"/>
-      </geometry>
-    </collision>
-  </link>
-  <link name="left_rear_wheel">
-    <inertial>
-      <mass value="${wheel_mass}"/>
-      <inertia ixx="0.062" ixy="0" ixz="0" iyy="0.093" iyz="0" izz="0.062"/>
-    </inertial>
-    <visual>
-      <material name="wheel_mat"/>
-      <origin xyz="0 0 0" rpy="1.5708 0 0"/>
-      <geometry>
-        <cylinder radius="${wheel_radius}" length="${wheel_length}"/>
-      </geometry>
-    </visual>
-    <collision>
-      <origin xyz="0 0 0" rpy="1.5708 0 0"/>
-      <geometry>
-        <cylinder radius="${wheel_radius}" length="${wheel_length}"/>
-      </geometry>
-    </collision>
-  </link>
-  <link name="right_front_wheel">
-    <inertial>
-      <mass value="${wheel_mass}"/>
-      <inertia ixx="0.062" ixy="0" ixz="0" iyy="0.093" iyz="0" izz="0.062"/>
-    </inertial>
-    <visual>
-      <material name="wheel_mat"/>
-      <origin xyz="0 0 0" rpy="1.5708 0 0"/>
-      <geometry>
-        <cylinder radius="${wheel_radius}" length="${wheel_length}"/>
-      </geometry>
-    </visual>
-    <collision>
-      <origin xyz="0 0 0" rpy="1.5708 0 0"/>
-      <geometry>
-        <cylinder radius="${wheel_radius}" length="${wheel_length}"/>
-      </geometry>
-    </collision>
-  </link>
-  <link name="right_rear_wheel">
-    <inertial>
-      <mass value="${wheel_mass}"/>
-      <inertia ixx="0.062" ixy="0" ixz="0" iyy="0.093" iyz="0" izz="0.062"/>
-    </inertial>
-    <visual>
-      <material name="wheel_mat"/>
-      <origin xyz="0 0 0" rpy="1.5708 0 0"/>
-      <geometry>
-        <cylinder radius="${wheel_radius}" length="${wheel_length}"/>
-      </geometry>
-    </visual>
-    <collision>
-      <origin xyz="0 0 0" rpy="1.5708 0 0"/>
-      <geometry>
-        <cylinder radius="${wheel_radius}" length="${wheel_length}"/>
-      </geometry>
-    </collision>
-  </link>
-<!-- TURNTABLES -->
-<link name="left_front_turntable">
-  <inertial>
-    <mass value="${turntable_mass}"/>
-    <inertia ixx="0.01" ixy="0" ixz="0" iyy="0.01" iyz="0" izz="0.01"/>
-  </inertial>
-  <visual>
-    <origin xyz="0 0 ${turntable_height/2}" rpy="0 0 0"/>
-    <geometry>
-      <cylinder radius="${turntable_radius}" length="${turntable_height}"/>
-    </geometry>
-  </visual>
-</link>
-<link name="left_rear_turntable">
-  <inertial>
-    <mass value="${turntable_mass}"/>
-    <inertia ixx="0.01" ixy="0" ixz="0" iyy="0.01" iyz="0" izz="0.01"/>
-  </inertial>
-  <visual>
-    <origin xyz="0 0 ${turntable_height/2}" rpy="0 0 0"/>
-    <geometry>
-      <cylinder radius="${turntable_radius}" length="${turntable_height}"/>
-    </geometry>
-  </visual>
-</link>
-<link name="right_front_turntable">
-  <inertial>
-    <mass value="${turntable_mass}"/>
-    <inertia ixx="0.01" ixy="0" ixz="0" iyy="0.01" iyz="0" izz="0.01"/>
-  </inertial>
-  <visual>
-    <origin xyz="0 0 ${turntable_height/2}" rpy="0 0 0"/>
-    <geometry>
-      <cylinder radius="${turntable_radius}" length="${turntable_height}"/>
-    </geometry>
-  </visual>
-</link>
-<link name="right_rear_turntable">
-  <inertial>
-    <mass value="${turntable_mass}"/>
-    <inertia ixx="0.01" ixy="0" ixz="0" iyy="0.01" iyz="0" izz="0.01"/>
-  </inertial>
-  <visual>
-    <origin xyz="0 0 ${turntable_height/2}" rpy="0 0 0"/>
-    <geometry>
-      <cylinder radius="${turntable_radius}" length="${turntable_height}"/>
-    </geometry>
-  </visual>
-</link>
-<!-- JOINTS -->
-<joint name="realsense_front_joint" type="fixed">
-  <parent link="realsense_front_link"/>
-  <child link="chassis"/>
-  <axis xyz="1 0 0"/>
-</joint>
-<joint name="suspension_diff_joint" type="continuous">
-  <parent link="chassis"/>
-  <child link="suspension_diff"/>
-  <axis xyz="0 1 0"/>
-</joint>
-<joint name="left_subchassis_hinge" type="continuous">
-  <parent link="suspension_diff"/>
-  <child link="left_subchassis"/>
-  <axis xyz="0 1 0"/>
-</joint>
-<joint name="right_subchassis_hinge" type="continuous">
-  <parent link="suspension_diff"/>
-  <child link="right_subchassis"/>
-  <axis xyz="0 1 0"/>
-</joint>
-<joint name="left_front_turntable_joint" type="continuous">
-  <parent link="left_subchassis"/>
-  <child link="left_front_turntable"/>
-  <origin xyz="$(eval ${wheel_spacing_x}/2) $(eval ${wheel_spacing_y}/2) ${subchassis_origin_z}" rpy="0 0 0"/>
-  <axis xyz="0 0 1"/>
-</joint>
-<joint name="left_rear_turntable_joint" type="continuous">
-  <parent link="left_subchassis"/>
-  <child link="left_rear_turntable"/>
-  <origin xyz="$(eval -${wheel_spacing_x}/2) $(eval ${wheel_spacing_y}/2) ${subchassis_origin_z}" rpy="0 0 0"/>
-  <axis xyz="0 0 1"/>
-</joint>
-<joint name="right_front_turntable_joint" type="continuous">
-  <parent link="right_subchassis"/>
-  <child link="right_front_turntable"/>
-  <origin xyz="$(eval ${wheel_spacing_x}/2) $(eval -${wheel_spacing_y}/2) ${subchassis_origin_z}" rpy="0 0 0"/>
-  <axis xyz="0 0 1"/>
-</joint>
-<joint name="right_rear_turntable_joint" type="continuous">
-  <parent link="right_subchassis"/>
-  <child link="right_rear_turntable"/>
-  <origin xyz="$(eval -${wheel_spacing_x}/2) $(eval -${wheel_spacing_y}/2) ${subchassis_origin_z}" rpy="0 0 0"/>
-  <axis xyz="0 0 1"/>
-</joint>
-<joint name="left_front_wheel_joint" type="continuous">
-  <parent link="left_front_turntable"/>
-  <child link="left_front_wheel"/>
-  <origin xyz="0 0 $(eval -${turntable_height}/2 - ${wheel_radius})" rpy="0 0 0"/>
-  <axis xyz="0 1 0"/>
-</joint>
-<joint name="left_rear_wheel_joint" type="continuous">
-  <parent link="left_rear_turntable"/>
-  <child link="left_rear_wheel"/>
-  <origin xyz="0 0 $(eval -${turntable_height}/2 - ${wheel_radius})" rpy="0 0 0"/>
-  <axis xyz="0 1 0"/>
-</joint>
-<joint name="right_front_wheel_joint" type="continuous">
-  <parent link="right_front_turntable"/>
-  <child link="right_front_wheel"/>
-  <origin xyz="0 0 $(eval -${turntable_height}/2 - ${wheel_radius})" rpy="0 0 0"/>
-  <axis xyz="0 1 0"/>
-</joint>
-<joint name="right_rear_wheel_joint" type="continuous">
-  <parent link="right_rear_turntable"/>
-  <child link="right_rear_wheel"/>
-  <origin xyz="0 0 $(eval -${turntable_height}/2 - ${wheel_radius})" rpy="0 0 0"/>
-  <axis xyz="0 1 0"/>
-</joint>
+<!--
+  Robot: orion_VI
+  Generated by: LinkForge v1.4.4
+  https://github.com/arounamounchili/linkforge
+  Date: 2026-08-10 13:27:38
+-->
+<robot xmlns:xacro="http://ros.org/xacro" name="orion_VI">
+  <!-- Links -->
+  <link name="base_link">
+    <inertial>
+      <origin xyz="0 -0.006868 0.003669" rpy="0 0 0" />
+      <mass value="20" />
+      <inertia ixx="0.807298" ixy="0" ixz="0" iyy="0.351972" iyz="0" izz="0.953009" />
+    </inertial>
+    <visual>
+      <origin xyz="0 -0.006868 0.323814" rpy="0 0 0" />
+      <geometry>
+        <mesh filename="package://orion_vi_description/urdf/meshes/base_link_visual.obj" />
+      </geometry>
+    </visual>
+    <collision>
+      <origin xyz="0 -0.006868 0.003669" rpy="0 0 0" />
+      <geometry>
+        <box size="0.3864 0.65 0.248753" />
+      </geometry>
+    </collision>
+  </link>
+  <link name="module_F">
+    <inertial>
+      <origin xyz="0.365016 -0.007428 0.00981" rpy="0 0 0" />
+      <mass value="5" />
+      <inertia ixx="0.081035" ixy="0" ixz="0" iyy="0.073194" iyz="0" izz="0.106243" />
+    </inertial>
+    <visual>
+      <origin xyz="0.365016 -0.007428 0.00981" rpy="0 0 0" />
+      <geometry>
+        <mesh filename="package://orion_vi_description/urdf/meshes/module_F_visual.obj" />
+      </geometry>
+    </visual>
+    <collision>
+      <origin xyz="0.365016 -0.007428 0.00981" rpy="0 0 0" />
+      <geometry>
+        <box size="0.343633 0.37 0.239965" />
+      </geometry>
+    </collision>
+  </link>
+  <link name="module_rear">
+    <inertial>
+      <origin xyz="0.027984 0.001017 0.004581" rpy="0 0 0" />
+      <mass value="5" />
+      <inertia ixx="0.081035" ixy="0" ixz="0" iyy="0.073194" iyz="0" izz="0.106243" />
+    </inertial>
+    <visual>
+      <origin xyz="0.027984 0.001017 0.004581" rpy="0 0 0" />
+      <geometry>
+        <mesh filename="package://orion_vi_description/urdf/meshes/module_rear_visual.obj" />
+      </geometry>
+    </visual>
+    <collision>
+      <origin xyz="0.027984 0.001017 0.004581" rpy="0 0 0" />
+      <geometry>
+        <box size="0.343633 0.37 0.239965" />
+      </geometry>
+    </collision>
+  </link>
+  <link name="realsense">
+    <inertial>
+      <origin xyz="-0.012527 0.000043 0" rpy="3.141593 0 1.570796" />
+      <mass value="0.075" />
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
File: src/orion_vi_description/urdf/sensors/bootlegsense.xacro (robot description, xacro)
@@ -1,9 +1,9 @@
 <?xml version="1.0"?>
 <robot xmlns:xacro="http://www.ros.org/wiki/xacro" >
-<xacro:macro name="add_realsense" params="suffix">
-    <gazebo reference="realsense_${suffix}_link">
-    <sensor name="realsense_d435i_${suffix}" type="rgbd_camera">
+<xacro:macro name="add_realsense">
+    <gazebo reference="realsense">
+    <sensor name="realsense_d435i" type="rgbd_camera">
         <update_rate>60</update_rate>
-        <topic>realsense_d435i_${suffix}</topic>
+        <topic>realsense_d435i</topic>
         <camera name="camera">
           <horizontal_fov>1.0472</horizontal_fov>
