Commit message: added the camera link as a root

File: src/orion_vi_description/urdf/orionVI_description.urdf.xacro (robot description, xacro)
@@ -52,5 +52,4 @@
   <xacro:property name="turntable_radius" value="$(eval ${subchassis_y}/2)"/>
   <xacro:property name="turntable_mass" value="1.0"/>
-  <!-- CHASSIS -->
   <!-- Materials -->
   <material name="wheel_mat">
@@ -63,4 +62,18 @@
     <color rgba="0.6431373 0.6431373 0.6431373 1.0"/>
   </material>
+  <!--CAMERA-->
+  <link name="camera">
+    <inertial>
+      <origin xyz="${chassis_x/2} 0 ${chassis_y+chassis_origin_z}" rpy="0 0 0"/>
+    </inertial>
+    <visual name="camera_visual">
+      <material name="chassis_mat"/>
+      <origin xyz="${chassis_x/2} 0 ${chassis_y+chassis_origin_z}" rpy="0 0 0"/>
+      <geometry>
+        <box size="0.01 0.02 0.01"/>
+      </geometry>
+    </visual>
+  </link>
+  <!-- CHASSIS -->
   <link name="chassis">
     <inertial>
@@ -258,20 +271,25 @@
   </visual>
 </link>
-  <!-- JOINTS -->
-  <joint name="suspension_diff_joint" type="continuous">
-    <parent link="chassis"/>
-    <child link="suspension_diff"/>
-    <axis xyz="0 1 0"/>
-  </joint>
-  <joint name="left_subchassis_hinge" type="continuous">
-    <parent link="suspension_diff"/>
-    <child link="left_subchassis"/>
-    <axis xyz="0 1 0"/>
-  </joint>
-  <joint name="right_subchassis_hinge" type="continuous">
-    <parent link="suspension_diff"/>
-    <child link="right_subchassis"/>
-    <axis xyz="0 1 0"/>
-  </joint>
+<!-- JOINTS -->
+<joint name="camera_joint" type="fixed">
+  <parent link="camera"/>
+  <child link="chassis"/>
+  <axis xyz="1 0 0"/>
+</joint>
+<joint name="suspension_diff_joint" type="continuous">
+  <parent link="chassis"/>
+  <child link="suspension_diff"/>
+  <axis xyz="0 1 0"/>
+</joint>
+<joint name="left_subchassis_hinge" type="continuous">
+  <parent link="suspension_diff"/>
+  <child link="left_subchassis"/>
+  <axis xyz="0 1 0"/>
+</joint>
+<joint name="right_subchassis_hinge" type="continuous">
+  <parent link="suspension_diff"/>
+  <child link="right_subchassis"/>
+  <axis xyz="0 1 0"/>
+</joint>
 <joint name="left_front_turntable_joint" type="continuous">
   <parent link="left_subchassis"/>

Commit message: fix: fixed camera link

File: src/orion_vi_description/urdf/orionVI_description.urdf.xacro (robot description, xacro)
@@ -64,12 +64,10 @@
   <!--CAMERA-->
   <link name="camera">
-    <inertial>
-      <origin xyz="${chassis_x/2} 0 ${chassis_y+chassis_origin_z}" rpy="0 0 0"/>
-    </inertial>
+    <origin xyz="${chassis_x/2} 0 ${(chassis_z+chassis_origin_z)/2}" rpy="0 0 0"/>
     <visual name="camera_visual">
       <material name="chassis_mat"/>
-      <origin xyz="${chassis_x/2} 0 ${chassis_y+chassis_origin_z}" rpy="0 0 0"/>
-      <geometry>
-        <box size="0.01 0.02 0.01"/>
+      <origin xyz="${chassis_x/2} 0 ${(chassis_z+chassis_origin_z)/2}" rpy="0 0 0"/>
+      <geometry>
+        <box size="0.1 0.2 0.1"/>
       </geometry>
     </visual>

Commit message: fix: updated rocker joint position

File: src/orion_vi_description/urdf/orionVI_description.urdf.xacro (robot description, xacro)
@@ -2,7 +2,7 @@
 <!--
   Robot: orion_VI
-  Generated by: LinkForge v1.4.4
+  Generated by: LinkForge v1.5.0
   https://github.com/arounamounchili/linkforge
-  Date: 2026-08-10 13:27:38
+  Date: 2026-08-12 17:38:24
 -->
 <robot xmlns:xacro="http://ros.org/xacro" name="orion_VI">
@@ -12,5 +12,5 @@
       <origin xyz="0 -0.006868 0.003669" rpy="0 0 0" />
       <mass value="20" />
-      <inertia ixx="0.807298" ixy="0" ixz="0" iyy="0.351972" iyz="0" izz="0.953009" />
+      <inertia ixx="3.333333" ixy="0" ixz="0" iyy="3.333333" iyz="0" izz="3.333333" />
     </inertial>
     <visual>
@@ -23,5 +23,5 @@
       <origin xyz="0 -0.006868 0.003669" rpy="0 0 0" />
       <geometry>
-        <box size="0.3864 0.65 0.248753" />
+        <mesh filename="package://orion_vi_description/urdf/meshes/base_link_collision.stl" />
       </geometry>
     </collision>
@@ -31,5 +31,5 @@
       <origin xyz="0.365016 -0.007428 0.00981" rpy="0 0 0" />
       <mass value="5" />
-      <inertia ixx="0.081035" ixy="0" ixz="0" iyy="0.073194" iyz="0" izz="0.106243" />
+      <inertia ixx="0.833333" ixy="0" ixz="0" iyy="0.833333" iyz="0" izz="0.833333" />
     </inertial>
     <visual>
@@ -42,5 +42,5 @@
       <origin xyz="0.365016 -0.007428 0.00981" rpy="0 0 0" />
       <geometry>
-        <box size="0.343633 0.37 0.239965" />
+        <mesh filename="package://orion_vi_description/urdf/meshes/module_F_collision.stl" />
       </geometry>
     </collision>
@@ -50,5 +50,5 @@
       <origin xyz="0.027984 0.001017 0.004581" rpy="0 0 0" />
       <mass value="5" />
-      <inertia ixx="0.081035" ixy="0" ixz="0" iyy="0.073194" iyz="0" izz="0.106243" />
+      <inertia ixx="0.833333" ixy="0" ixz="0" iyy="0.833333" iyz="0" izz="0.833333" />
     </inertial>
     <visual>
@@ -61,5 +61,5 @@
       <origin xyz="0.027984 0.001017 0.004581" rpy="0 0 0" />
       <geometry>
-        <box size="0.343633 0.37 0.239965" />
+        <mesh filename="package://orion_vi_description/urdf/meshes/module_rear_collision.stl" />
       </geometry>
     </collision>
@@ -67,10 +67,10 @@
   <link name="realsense">
     <inertial>
+      <origin xyz="-0.012527 0.000043 0" rpy="0 0 0" />
+      <mass value="0.075" />
+      <inertia ixx="0.0125" ixy="0" ixz="0" iyy="0.0125" iyz="0" izz="0.0125" />
+    </inertial>
+    <visual>
       <origin xyz="-0.012527 0.000043 0" rpy="3.141593 0 1.570796" />
-      <mass value="0.075" />
-      <inertia ixx="0.000008" ixy="0" ixz="0" iyy="0.000054" iyz="0" izz="0.000054" />
-    </inertial>
-    <visual>
-      <origin xyz="-0.012527 0.000043 0" rpy="3.141593 0 1.570796" />
       <geometry>
         <mesh filename="package://orion_vi_description/urdf/meshes/realsense_visual.obj" />
@@ -78,7 +78,7 @@
     </visual>
     <collision>
-      <origin xyz="-0.012527 0.000043 0" rpy="3.141593 0 1.570796" />
-      <geometry>
-        <box size="0.089914 0.025055 0.025" />
+      <origin xyz="-0.012527 0.000043 0" rpy="0 0 0" />
+      <geometry>
+        <mesh filename="package://orion_vi_description/urdf/meshes/realsense_collision.stl" />
       </geometry>
     </collision>
@@ -124,5 +124,5 @@
   <link name="turntable_F_L">
     <inertial>
-      <origin xyz="0.000987 -0.020984 0.001439" rpy="0 0 0" />
+      <origin xyz="0.000734 -0.020984 -0.009735" rpy="0 0 0" />
       <mass value="2" />
       <inertia ixx="0.333333" ixy="0" ixz="0" iyy="0.333333" iyz="0" izz="0.333333" />
@@ -134,10 +134,4 @@
       </geometry>
     </visual>
-    <collision>
-      <origin xyz="0.000987 -0.020984 0.001439" rpy="0 0 0" />
-      <geometry>
-        <mesh filename="package://orion_vi_description/urdf/meshes/turntable_F_L_collision.stl" />
-      </geometry>
-    </collision>
   </link>
   <link name="turntable_F_R">
@@ -201,7 +195,7 @@
   <link name="wheel_F_R">
     <inertial>
-      <origin xyz="0 0 0" rpy="1.570796 0 0" />
-      <mass value="5" />
-      <inertia ixx="0.081575" ixy="0" ixz="0" iyy="0.081575" iyz="0" izz="0.128865" />
+      <origin xyz="0 0 0" rpy="0 0 0" />
+      <mass value="5" />
+      <inertia ixx="0.833333" ixy="0" ixz="0" iyy="0.833333" iyz="0" izz="0.833333" />
     </inertial>
     <visual>
@@ -212,7 +206,7 @@
     </visual>
     <collision>
-      <origin xyz="0 0 0" rpy="1.570796 0 0" />
-      <geometry>
-        <cylinder radius="0.227037" length="0.202838" />
+      <origin xyz="0 0 0" rpy="0 0 0" />
+      <geometry>
+        <mesh filename="package://orion_vi_description/urdf/meshes/wheel_F_R_collision.stl" />
       </geometry>
     </collision>
@@ -220,7 +214,7 @@
   <link name="wheel_R_L">
     <inertial>
-      <origin xyz="0 0 0" rpy="1.570796 0 0" />
-      <mass value="5" />
-      <inertia ixx="0.081575" ixy="0" ixz="0" iyy="0.081575" iyz="0" izz="0.128865" />
+      <origin xyz="0 0 0" rpy="0 0 0" />
+      <mass value="5" />
+      <inertia ixx="0.833333" ixy="0" ixz="0" iyy="0.833333" iyz="0" izz="0.833333" />
     </inertial>
     <visual>
@@ -231,7 +225,7 @@
     </visual>
     <collision>
-      <origin xyz="0 0 0" rpy="1.570796 0 0" />
-      <geometry>
-        <cylinder radius="0.227037" length="0.202838" />
+      <origin xyz="0 0 0" rpy="0 0 0" />
+      <geometry>
+        <mesh filename="package://orion_vi_description/urdf/meshes/wheel_R_L_collision.stl" />
       </geometry>
     </collision>
@@ -239,7 +233,7 @@
   <link name="wheel_R_R">
     <inertial>
-      <origin xyz="0 0 0" rpy="1.570796 0 0" />
-      <mass value="5" />
-      <inertia ixx="0.081575" ixy="0" ixz="0" iyy="0.081575" iyz="0" izz="0.128865" />
+      <origin xyz="0 0 0" rpy="0 0 0" />
+      <mass value="5" />
+      <inertia ixx="0.833333" ixy="0" ixz="0" iyy="0.833333" iyz="0" izz="0.833333" />
     </inertial>
     <visual>
@@ -250,7 +244,7 @@
     </visual>
     <collision>
-      <origin xyz="0 0 0" rpy="1.570796 0 0" />
-      <geometry>
-        <cylinder radius="0.227037" length="0.202838" />
+      <origin xyz="0 0 0" rpy="0 0 0" />
+      <geometry>
+        <mesh filename="package://orion_vi_description/urdf/meshes/wheel_R_R_collision.stl" />
       </geometry>
     </collision>

Commit message: fix: fixed turntable joint axis

File: src/orion_vi_description/urdf/orionVI_description.urdf.xacro (robot description, xacro)
@@ -4,5 +4,5 @@
   Generated by: LinkForge v1.5.0
   https://github.com/arounamounchili/linkforge
-  Date: 2026-08-12 17:38:24
+  Date: 2026-08-12 22:17:32
 -->
 <robot xmlns:xacro="http://ros.org/xacro" name="orion_VI">
@@ -290,5 +290,5 @@
     <parent link="rocker_R" />
     <child link="turntable_F_R" />
-    <axis xyz="0 1 0" />
+    <axis xyz="0 0 1" />
     <limit effort="10" velocity="1" lower="-3.141593" upper="3.141593" />
   </joint>
@@ -297,5 +297,5 @@
     <parent link="rocker_L" />
     <child link="turntable_R_L" />
-    <axis xyz="0 1 0" />
+    <axis xyz="0 0 1" />
     <limit effort="10" velocity="1" lower="-3.141593" upper="3.141593" />
   </joint>
@@ -304,5 +304,5 @@
     <parent link="rocker_R" />
     <child link="turntable_R_R" />
-    <axis xyz="0 1 0" />
+    <axis xyz="0 0 1" />
     <limit effort="10" velocity="1" lower="-3.141593" upper="3.141593" />
   </joint>
