Commit message: fix: camera_link xarco description remove duplicate verticies

File: src/orion_vi_description/urdf/orionVI_description.urdf.xacro (robot description, xacro)
@@ -2,18 +2,12 @@
 <!--
   Robot: orion_VI
-  Generated by: LinkForge v1.5.0
+  Generated by: LinkForge
   https://github.com/arounamounchili/linkforge
-  Date: 2026-08-12 22:17:32
 -->
-<robot xmlns:xacro="http://ros.org/xacro" name="orion_VI">
+<robot xmlns:xacro="http://ros.org/wiki/xacro" name="orion_VI">
   <!-- Links -->
   <link name="base_link">
-    <inertial>
-      <origin xyz="0 -0.006868 0.003669" rpy="0 0 0" />
-      <mass value="20" />
-      <inertia ixx="3.333333" ixy="0" ixz="0" iyy="3.333333" iyz="0" izz="3.333333" />
-    </inertial>
-    <visual>
-      <origin xyz="0 -0.006868 0.323814" rpy="0 0 0" />
+    <visual>
+      <origin xyz="-1.490116e-08 -0.006868 0.323814" rpy="0 0 0" />
       <geometry>
         <mesh filename="package://orion_vi_description/urdf/meshes/base_link_visual.obj" />
@@ -21,5 +15,5 @@
     </visual>
     <collision>
-      <origin xyz="0 -0.006868 0.003669" rpy="0 0 0" />
+      <origin xyz="-1.490116e-08 -0.006868 0.003669" rpy="0 0 0" />
       <geometry>
         <mesh filename="package://orion_vi_description/urdf/meshes/base_link_collision.stl" />
@@ -27,58 +21,64 @@
     </collision>
   </link>
-  <link name="module_F">
-    <inertial>
-      <origin xyz="0.365016 -0.007428 0.00981" rpy="0 0 0" />
-      <mass value="5" />
-      <inertia ixx="0.833333" ixy="0" ixz="0" iyy="0.833333" iyz="0" izz="0.833333" />
-    </inertial>
-    <visual>
-      <origin xyz="0.365016 -0.007428 0.00981" rpy="0 0 0" />
-      <geometry>
-        <mesh filename="package://orion_vi_description/urdf/meshes/module_F_visual.obj" />
-      </geometry>
-    </visual>
-    <collision>
-      <origin xyz="0.365016 -0.007428 0.00981" rpy="0 0 0" />
-      <geometry>
-        <mesh filename="package://orion_vi_description/urdf/meshes/module_F_collision.stl" />
-      </geometry>
-    </collision>
-  </link>
-  <link name="module_rear">
-    <inertial>
-      <origin xyz="0.027984 0.001017 0.004581" rpy="0 0 0" />
-      <mass value="5" />
-      <inertia ixx="0.833333" ixy="0" ixz="0" iyy="0.833333" iyz="0" izz="0.833333" />
-    </inertial>
-    <visual>
-      <origin xyz="0.027984 0.001017 0.004581" rpy="0 0 0" />
-      <geometry>
-        <mesh filename="package://orion_vi_description/urdf/meshes/module_rear_visual.obj" />
-      </geometry>
-    </visual>
-    <collision>
-      <origin xyz="0.027984 0.001017 0.004581" rpy="0 0 0" />
-      <geometry>
-        <mesh filename="package://orion_vi_description/urdf/meshes/module_rear_collision.stl" />
-      </geometry>
-    </collision>
-  </link>
-  <link name="realsense">
-    <inertial>
-      <origin xyz="-0.012527 0.000043 0" rpy="0 0 0" />
+  <link name="camera_link">
+    <inertial>
+      <origin xyz="-0.012527 4.300475e-05 0" rpy="0 0 0" />
       <mass value="0.075" />
       <inertia ixx="0.0125" ixy="0" ixz="0" iyy="0.0125" iyz="0" izz="0.0125" />
     </inertial>
     <visual>
-      <origin xyz="-0.012527 0.000043 0" rpy="3.141593 0 1.570796" />
-      <geometry>
-        <mesh filename="package://orion_vi_description/urdf/meshes/realsense_visual.obj" />
-      </geometry>
-    </visual>
-    <collision>
-      <origin xyz="-0.012527 0.000043 0" rpy="0 0 0" />
-      <geometry>
-        <mesh filename="package://orion_vi_description/urdf/meshes/realsense_collision.stl" />
+      <origin xyz="-0.012527 4.300494e-05 0" rpy="3.141593 4.371138e-08 1.570796" />
+      <geometry>
+        <mesh filename="package://orion_vi_description/urdf/meshes/camera_link_visual.obj" />
+      </geometry>
+    </visual>
+    <collision>
+      <origin xyz="-0.012527 4.300475e-05 0" rpy="0 0 0" />
+      <geometry>
+        <mesh filename="package://orion_vi_description/urdf/meshes/camera_link_collision.stl" />
+      </geometry>
+    </collision>
+  </link>
+  <link name="main_body">
+    <inertial>
+      <mass value="20" />
+      <inertia ixx="1" ixy="0" ixz="0" iyy="1" iyz="0" izz="1" />
+    </inertial>
+  </link>
+  <link name="module_F">
+    <inertial>
+      <origin xyz="0.365016 -0.007428 0.00981" rpy="0 0 0" />
+      <mass value="5" />
+      <inertia ixx="0.833333" ixy="0" ixz="0" iyy="0.833333" iyz="0" izz="0.833333" />
+    </inertial>
+    <visual>
+      <origin xyz="0.365016 -0.007428 0.00981" rpy="0 0 0" />
+      <geometry>
+        <mesh filename="package://orion_vi_description/urdf/meshes/module_F_visual.obj" />
+      </geometry>
+    </visual>
+    <collision>
+      <origin xyz="0.365016 -0.007428 0.00981" rpy="0 0 0" />
+      <geometry>
+        <mesh filename="package://orion_vi_description/urdf/meshes/module_F_collision.stl" />
+      </geometry>
+    </collision>
+  </link>
+  <link name="module_R">
+    <inertial>
+      <origin xyz="0.027984 0.001017 0.004581" rpy="0 0 0" />
+      <mass value="5" />
+      <inertia ixx="0.833333" ixy="0" ixz="0" iyy="0.833333" iyz="0" izz="0.833333" />
+    </inertial>
+    <visual>
+      <origin xyz="0.027984 0.001017 0.004581" rpy="0 0 0" />
+      <geometry>
+        <mesh filename="package://orion_vi_description/urdf/meshes/module_R_visual.obj" />
+      </geometry>
+    </visual>
+    <collision>
+      <origin xyz="0.027984 0.001017 0.004581" rpy="0 0 0" />
+      <geometry>
+        <mesh filename="package://orion_vi_description/urdf/meshes/module_R_collision.stl" />
       </geometry>
     </collision>
@@ -86,10 +86,10 @@
   <link name="rocker_L">
     <inertial>
-      <origin xyz="0 0.061026 -0.047943" rpy="0 0 0" />
+      <origin xyz="-5.960464e-08 0.061026 -0.047943" rpy="0 0 0" />
       <mass value="15" />
       <inertia ixx="2.5" ixy="0" ixz="0" iyy="2.5" iyz="0" izz="2.5" />
     </inertial>
     <visual>
-      <origin xyz="0 0 -0.047943" rpy="0 0 0" />
+      <origin xyz="-5.960464e-08 2.980232e-08 -0.047943" rpy="0 0 0" />
       <geometry>
         <mesh filename="package://orion_vi_description/urdf/meshes/rocker_L_visual.obj" />
@@ -97,5 +97,5 @@
     </visual>
     <collision>
-      <origin xyz="0 0.061026 -0.047943" rpy="0 0 0" />
+      <origin xyz="-5.960464e-08 0.061026 -0.047943" rpy="0 0 0" />
       <geometry>
         <mesh filename="package://orion_vi_description/urdf/meshes/rocker_L_collision.stl" />
@@ -105,10 +105,10 @@
   <link name="rocker_R">
     <inertial>
-      <origin xyz="0 -0.058921 -0.047943" rpy="0 0 0" />
+      <origin xyz="-5.960464e-08 -0.058921 -0.047943" rpy="0 0 0" />
       <mass value="15" />
       <inertia ixx="2.5" ixy="0" ixz="0" iyy="2.5" iyz="0" izz="2.5" />
     </inertial>
     <visual>
-      <origin xyz="0 0 -0.047943" rpy="0 0 0" />
+      <origin xyz="-2.980232e-08 -2.980232e-08 -0.047943" rpy="0 0 0" />
       <geometry>
         <mesh filename="package://orion_vi_description/urdf/meshes/rocker_R_visual.obj" />
@@ -116,5 +116,5 @@
     </visual>
     <collision>
-      <origin xyz="0 -0.058921 -0.047943" rpy="0 0 0" />
+      <origin xyz="-5.960464e-08 -0.058921 -0.047943" rpy="0 0 0" />
       <geometry>
         <mesh filename="package://orion_vi_description/urdf/meshes/rocker_R_collision.stl" />
@@ -176,5 +176,24 @@
   <link name="wheel_F_L">
     <inertial>
-      <origin xyz="0 0 0" rpy="0 0 0" />
+      <origin xyz="-2.980232e-08 0 0" rpy="0 0 0" />
+      <mass value="5" />
+      <inertia ixx="0.833333" ixy="0" ixz="0" iyy="0.833333" iyz="0" izz="0.833333" />
+    </inertial>
+    <visual>
+      <origin xyz="-3.278255e-07 -0.00155 -4.917383e-07" rpy="0 0 0" />
+      <geometry>
+        <mesh filename="package://orion_vi_description/urdf/meshes/wheel_F_L_visual.obj" />
+      </geometry>
+    </visual>
+    <collision>
+      <origin xyz="-2.980232e-08 0 0" rpy="0 0 0" />
+      <geometry>
+        <mesh filename="package://orion_vi_description/urdf/meshes/wheel_F_L_collision.stl" />
+      </geometry>
+    </collision>
+  </link>
+  <link name="wheel_F_R">
+    <inertial>
+      <origin xyz="-2.980232e-08 0 1.490116e-08" rpy="0 0 0" />
       <mass value="5" />
       <inertia ixx="0.833333" ixy="0" ixz="0" iyy="0.833333" iyz="0" izz="0.833333" />
@@ -183,28 +202,9 @@
       <origin xyz="0 -0.00155 0" rpy="0 0 0" />
       <geometry>
-        <mesh filename="package://orion_vi_description/urdf/meshes/wheel_F_L_visual.obj" />
-      </geometry>
-    </visual>
-    <collision>
-      <origin xyz="0 0 0" rpy="0 0 0" />
-      <geometry>
-        <mesh filename="package://orion_vi_description/urdf/meshes/wheel_F_L_collision.stl" />
-      </geometry>
-    </collision>
-  </link>
-  <link name="wheel_F_R">
-    <inertial>
-      <origin xyz="0 0 0" rpy="0 0 0" />
-      <mass value="5" />
-      <inertia ixx="0.833333" ixy="0" ixz="0" iyy="0.833333" iyz="0" izz="0.833333" />
-    </inertial>
-    <visual>
-      <origin xyz="0 -0.00155 0" rpy="0 0 0" />
-      <geometry>
         <mesh filename="package://orion_vi_description/urdf/meshes/wheel_F_R_visual.obj" />
       </geometry>
     </visual>
     <collision>
-      <origin xyz="0 0 0" rpy="0 0 0" />
+      <origin xyz="-2.980232e-08 0 1.490116e-08" rpy="0 0 0" />
       <geometry>
         <mesh filename="package://orion_vi_description/urdf/meshes/wheel_F_R_collision.stl" />
@@ -214,5 +214,5 @@
   <link name="wheel_R_L">
     <inertial>
-      <origin xyz="0 0 0" rpy="0 0 0" />
+      <origin xyz="0 -2.980232e-08 0" rpy="0 0 0" />
       <mass value="5" />
       <inertia ixx="0.833333" ixy="0" ixz="0" iyy="0.833333" iyz="0" izz="0.833333" />
@@ -225,5 +225,5 @@
     </visual>
     <collision>
-      <origin xyz="0 0 0" rpy="0 0 0" />
+      <origin xyz="0 -2.980232e-08 0" rpy="0 0 0" />
       <geometry>
         <mesh filename="package://orion_vi_description/urdf/meshes/wheel_R_L_collision.stl" />
@@ -233,5 +233,5 @@
   <link name="wheel_R_R">
     <inertial>
-      <origin xyz="0 0 0" rpy="0 0 0" />
+      <origin xyz="0 -2.980232e-08 1.490116e-08" rpy="0 0 0" />
       <mass value="5" />
       <inertia ixx="0.833333" ixy="0" ixz="0" iyy="0.833333" iyz="0" izz="0.833333" />
@@ -244,5 +244,5 @@
     </visual>
     <collision>
-      <origin xyz="0 0 0" rpy="0 0 0" />
+      <origin xyz="0 -2.980232e-08 1.490116e-08" rpy="0 0 0" />
       <geometry>
         <mesh filename="package://orion_vi_description/urdf/meshes/wheel_R_R_collision.stl" />
@@ -251,8 +251,14 @@
   </link>
   <!-- Joints -->
-  <joint name="base_link_joint" type="fixed">
-    <origin xyz="0.13 0 -0.6" rpy="0 0 0" />
-    <parent link="realsense" />
-    <child link="base_link" />
+  <joint name="camera_link_joint" type="fixed">
+    <origin xyz="-0.13 -2.980233e-08 0.6" rpy="0 0 0" />
+    <parent link="base_link" />
+    <child link="camera_link" />
+  </joint>
+  <joint name="main_body_joint" type="revolute">
+    <parent link="base_link" />
+    <child link="main_body" />
+    <axis xyz="0 0 1" />
+    <limit effort="10" velocity="1" lower="-3.141593" upper="3.141593" />
   </joint>
   <joint name="module_F_joint" type="fixed">
@@ -263,8 +269,8 @@
     <origin xyz="-0.393 -0.008446 0.005229" rpy="0 0 0" />
     <parent link="base_link" />
-    <child link="module_rear" />
+    <child link="module_R" />
   </joint>
   <joint name="rocker_L_joint" type="revolute">
-    <origin xyz="0 0.362582 0.141757" rpy="0 0 0" />
+    <origin xyz="-2.682209e-07 0.362582 0.141757" rpy="0 0 0" />
     <parent link="base_link" />
     <child link="rocker_L" />
@@ -273,5 +279,5 @@
   </joint>
   <joint name="rocker_R_joint" type="revolute">
-    <origin xyz="0 -0.362582 0.141757" rpy="0 0 0" />
+    <origin xyz="-2.682209e-07 -0.362582 0.141757" rpy="0 0 0" />
     <parent link="base_link" />
     <child link="rocker_R" />
@@ -307,31 +313,31 @@
     <limit effort="10" velocity="1" lower="-3.141593" upper="3.141593" />
   </joint>
-  <joint name="wheel_F_L_joint" type="revolute">
+  <joint name="wheel_F_L_joint" type="continuous">
     <origin xyz="0.000734 -0.022534 -0.106372" rpy="0 0 0" />
     <parent link="turntable_F_L" />
     <child link="wheel_F_L" />
     <axis xyz="0 1 0" />
-    <limit effort="10" velocity="1" lower="-3.141593" upper="3.141593" />
-  </joint>
-  <joint name="wheel_F_R_joint" type="revolute">
-    <origin xyz="-0.000733 0.022534 -0.106372" rpy="0 0 0" />
+    <limit effort="10" velocity="1" lower="0" upper="0" />
+  </joint>
+  <joint name="wheel_F_R_joint" type="continuous">
+    <origin xyz="-0.000734 0.022534 -0.106372" rpy="0 0 0" />
     <parent link="turntable_F_R" />
     <child link="wheel_F_R" />
     <axis xyz="0 1 0" />
-    <limit effort="10" velocity="1" lower="-3.141593" upper="3.141593" />
-  </joint>
-  <joint name="wheel_R_L_joint" type="revolute">
+    <limit effort="10" velocity="1" lower="0" upper="0" />
+  </joint>
+  <joint name="wheel_R_L_joint" type="continuous">
     <origin xyz="0.000885 -0.024106 -0.10682" rpy="0 0 0" />
     <parent link="turntable_R_L" />
     <child link="wheel_R_L" />
     <axis xyz="0 1 0" />
-    <limit effort="10" velocity="1" lower="-3.141593" upper="3.141593" />
-  </joint>
-  <joint name="wheel_R_R_joint" type="revolute">
+    <limit effort="10" velocity="1" lower="0" upper="0" />
+  </joint>
+  <joint name="wheel_R_R_joint" type="continuous">
     <origin xyz="-0.000571 0.024106 -0.10682" rpy="0 0 0" />
     <parent link="turntable_R_R" />
     <child link="wheel_R_R" />
     <axis xyz="0 1 0" />
-    <limit effort="10" velocity="1" lower="-3.141593" upper="3.141593" />
+    <limit effort="10" velocity="1" lower="0" upper="0" />
   </joint>
 </robot>
